File: fet-module/fet-module.kicad_pcb (KiCad board)
At the start: 2 copper layers, 80 x 22 mm, 31 parts

Commit message: finish everything
Parts:
- removed R1: 10kΩ, Resistor_SMD:R_0603_1608Metric_Pad0.98x0.95mm_HandSolder
Routing:
- net Net-(U4-4A_(In)): track 27.2 -> 25.0 mm, vias 1 -> 0
Other:
- board text removed: "A: 1101"
