File: fet-module/fet-module.kicad_sch (KiCad schematic)
At the start: 29 parts, among them Q1 AOD4184A, Q2 AOD4184A, Q3 AOD4184A, Q4 AOD4184A

Commit message: finish everything
Parts:
- removed R1: 10kΩ, PCM_JLCPCB:R_0402, symbol PCM_JLCPCB-Resistors:0402,10kΩ
Other:
- note removed: "Address 1101"
