File: neo-module/neo-module.kicad_pcb (KiCad board)
At the start: 2 copper layers, 80 x 22 mm, 19 parts

Commit message: finish everything
Parts:
- removed R5: 10kΩ, Resistor_SMD:R_0603_1608Metric_Pad0.98x0.95mm_HandSolder
Routing:
- net Net-(U1-GP2): track 26.9 -> 23.4 mm, vias 1 -> 0
Other:
- board text removed: "A: 1011"
