File: neo-module/neo-module.kicad_sch (KiCad schematic)
At the start: 13 parts

Commit message: finish everything
Parts:
- removed R5: 10kΩ, PCM_JLCPCB:R_0402, symbol PCM_JLCPCB-Resistors:0402,10kΩ
Other:
- note removed: "Address 1011"
