File: oled-panel/oled-panel.kicad_pcb (KiCad board)
At the start: 2 copper layers, 52 x 38 mm, 12 parts

Commit message: finish everything
Other:
- board text added: "ProjectDMX Display v1 projectdmx.com"
Changed lines of the file:
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@@
 			(drillshape 0)
 			(scaleselection 1)
-			(outputdirectory "E:/Downloads/")
+			(outputdirectory "E:/Projects/ProjectDMX/display/")
 		)
 	)
@@
 		(layer "Edge.Cuts")
 	)
+	(gr_text "ProjectDMX Display v1\nprojectdmx.com"
+		(at 118 72 270)
+		(layer "F.SilkS")
+		(effects
+			(font
+				(size 1 1)
+				(thickness 0.15)
+			)
+		)
+	)
 	(segment
