File: relay-module/relay-module.kicad_sch (KiCad schematic)
At the start: 15 parts, among them K1 SRD-05VDC-SL-C, Q1 S8050, Q2 PC817X2NSZ9F, Q3 PC817X2NSZ9F

Commit message: add fog relay module
Parts:
- added C4: C, Imported:PHE840EB6100KB05R17, symbol Device:C
- added R4: R, Imported:FMP100JR-52-100R, symbol Device:R
- added R6: 10kΩ, Capacitor_SMD:C_0603_1608Metric_Pad1.08x0.95mm_HandSolder, symbol PCM_JLCPCB-Resistors:0402,10kΩ
- added U4: ~, ProjectDMX:DMX Alt JST, symbol ProjectDMX:Fog Out
- C1, C2, C3: footprint PCM_JLCPCB:C_0402 -> Capacitor_SMD:C_0603_1608Metric_Pad1.08x0.95mm_HandSolder
- D1: footprint PCM_JLCPCB:D_SMA -> Imported:1N4148W
- D2: footprint PCM_JLCPCB:D_SMA -> Imported:S1M
- K1: footprint SRD -> Imported:G5LE_14_DC5
- Q1: footprint PCM_JLCPCB:Q_SOT-23 -> Imported:S8050
- Q2, Q3: footprint DIP762W60P254L460H450Q4N -> Imported:PC817X2NSZ9F
- R1: footprint PCM_JLCPCB:R_0402 -> Imported:354047KFT
- R2, R3, R5: footprint PCM_JLCPCB:R_0402 -> Capacitor_SMD:C_0603_1608Metric_Pad1.08x0.95mm_HandSolder
- U2: footprint (none) -> ProjectDMX:Vert Terminal Block p3
Connections:
- net 5V: now also D1.1, K1.2 (C1)
- net GND: now also Q1.2 (E), R6.1; no longer D1.1, K1.2 (C1), Q1.1 (B)
- net at D2.2, Q2.2 (CATHODE), U2.2 (Neutral): now also U4.2 (Neutral); no longer K1.1 (COM)
- net at K1.4 (NO), U2.3 (Pump): now also C4.2, U4.3 (Pump)
- net at R3.1: now also Q1.1 (B), R6.2; no longer Q1.2 (E)
- net at R1.1, U2.1 (Hot): now also K1.1 (COM), R4.2, U4.1 (Hot)
- new net: C4.1, R4.1
Other:
- note added: "S1M 1000v"
- note added: "Use pico pullup"
- moved on the sheet: C1, C2, C3, D1, D2, K1, Q1, Q2, Q3, R1, R2, R3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

Commit message: finish everything
Parts:
- removed R5: 10kΩ, Capacitor_SMD:C_0603_1608Metric_Pad1.08x0.95mm_HandSolder, symbol PCM_JLCPCB-Resistors:0402,10kΩ
Other:
- note removed: "Address 1110"
