File: rfid-module/rfid-module.kicad_sch (KiCad schematic)
At the start: 60 parts, among them IC1 MCP23017-E_SO, Q1 BSS138, Q2 BSS138

Commit message: finish everything
Other:
- note removed: "Address 1111"
Changed lines of the file:
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@@
 	(paper "A4")
-	(rectangle
-		(start 238.76 97.79)
-		(end 246.888 123.19)
-		(stroke
-			(width 0)
-			(type default)
-		)
-		(fill
-			(type none)
-		)
-	)
 	(rectangle
 		(start 193.04 17.78)
@@
 		)
 	)
-	(text "Address\n1111\n"
-		(exclude_from_sim no)
-		(at 239.268 95.25 0)
-		(effects
-			(font
-				(size 1.27 1.27)
-			)
-			(justify left)
-		)
-	)
 	(junction
 		(at 60.96 109.22)
@@
 	(wire
 		(pts
-			(xy 237.49 121.92) (xy 257.81 121.92)
-		)
-		(stroke
-			(width 0)
-			(type default)
-		)
-	)
-	(wire
-		(pts
 			(xy 248.92 129.54) (xy 257.81 129.54)
 		)
@@
 		)
 		(stroke
+			(width 0)
+			(type default)
+		)
+	)
+	(wire
+		(pts
+			(xy 240.03 121.92) (xy 257.81 121.92)
+		)
+		(stroke
