File: rfid-module/rfid-module.kicad_pcb (KiCad board)
At the start: 2 copper layers, 80 x 22 mm, 38 parts, among them IC1 MCP23017-E_SO, Q1 BSS138, Q2 BSS138

Commit message: small changes
Parts:
- moved Q2 1.38 mm to (168.1, 92.0)
Routing:
- net Net-(Q2-S): track 71.0 -> 69.6 mm
- net 3V3: track 87.6 -> 86.6 mm
- net Net-(IC1-SCL): track 25.9 -> 25.1 mm
Changed lines of the file:
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@@
 		(tags "SOT TO_SOT_SMD")
 		(property "Reference" "Q1"
-			(at -2.9375 0.05 0)
+			(at 1.931649 -1.020569 0)
 			(layer "F.SilkS")
 			(effects
@@
 	(footprint "Package_TO_SOT_SMD:SOT-23"
 		(layer "F.Cu")
-		(at 169.4375 92)
+		(at 168.0625 92)
 		(descr "SOT, 3 Pin (JEDEC TO-236 Var AB https://www.jedec.org/document_search?search_api_views_fulltext=TO-236), generated with kicad-footprint-generator ipc_gullwing_generator.py")
 		(tags "SOT TO_SOT_SMD")
 		(property "Reference" "Q2"
-			(at -2.9375 0.05 0)
+			(at 1.9375 -1 0)
 			(layer "F.SilkS")
 			(effects
@@
 	)
 	(segment
-		(start 175.25 97.827)
-		(end 175.25 97.75)
+		(start 175.25 97.75)
+		(end 171 93.5)
 		(width 0.25)
 		(layer "B.Cu")
@@
 	)
 	(segment
-		(start 175.25 97.75)
-		(end 171.549 94.049)
+		(start 171 93.5)
+		(end 171 88.675)
 		(width 0.25)
 		(layer "B.Cu")
@@
 	)
 	(segment
-		(start 171.549 89.224)
+		(start 171 88.675)
 		(end 170.375 88.05)
 		(width 0.25)
@@
 	)
 	(segment
-		(start 171.549 94.049)
-		(end 171.549 89.224)
+		(start 175.25 97.827)
+		(end 175.25 97.75)
 		(width 0.25)
 		(layer "B.Cu")
@@
 	)
 	(via
-		(at 170.375 92)
+		(at 169 92)
 		(size 0.6)
 		(drill 0.3)
@@
 	)
 	(segment
-		(start 170.375 94.375)
-		(end 170.375 92)
+		(start 170.375 93.375)
+		(end 170.375 94.375)
 		(width 0.25)
 		(layer "B.Cu")
@@
 	)
 	(segment
-		(start 170.375 92)
+		(start 169 92)
 		(end 164.4125 92)
 		(width 0.25)
@@
 	)
 	(segment
+		(start 170.375 94.375)
+		(end 174.452 98.452)
+		(width 0.25)
+		(layer "B.Cu")
+		(net 22)
+	)
+	(segment
 		(start 174.452 98.452)
-		(end 170.375 94.375)
+		(end 176.029533 98.452)
 		(width 0.25)
 		(layer "B.Cu")
@@
 	)
 	(segment
-		(start 176.029533 98.452)
-		(end 174.452 98.452)
+		(start 169 92)
+		(end 170.375 93.375)
 		(width 0.25)
 		(layer "B.Cu")
@@
 	)
 	(segment
+		(start 164.675 93.5)
+		(end 164.675 96.5)
+		(width 0.5)
+		(layer "F.Cu")
+		(net 27)
+	)
+	(segment
 		(start 109.5875 85.5)
 		(end 109.5875 87)
@@
 	)
 	(segment
+		(start 167.3115 89.8615)
+		(end 167.125 90.048)
+		(width 0.5)
+		(layer "F.Cu")
+		(net 27)
+	)
+	(segment
 		(start 167.3115 88.2885)
 		(end 167.3115 89.8615)
@@
 	)
 	(segment
-		(start 167.3115 89.8615)
-		(end 168.5 91.05)
-		(width 0.5)
-		(layer "F.Cu")
-		(net 27)
-	)
-	(segment
-		(start 164.675 94.875)
-		(end 168.5 91.05)
+		(start 112.507152 90.32)
+		(end 114.5 92.312848)
 		(width 0.5)
 		(layer "F.Cu")
@@
 	)
 	(segment
-		(start 112.507152 90.32)
-		(end 114.5 92.312848)
+		(start 167.125 91.05)
+		(end 164.675 93.5)
 		(width 0.5)
 		(layer "F.Cu")
@@
 	)
 	(segment
-		(start 164.675 94.875)
-		(end 164.675 96.5)
+		(start 167.125 90.048)
+		(end 167.125 91.05)
 		(width 0.5)
 		(layer "F.Cu")
@@
 	)
 	(via
-		(at 168.5 92.95)
+		(at 167.125 92.95)
 		(size 0.6)
 		(drill 0.3)
@@
 	)
 	(segment
-		(start 163.55 92.95)
-		(end 163.5 93)
-		(width 0.25)
-		(layer "B.Cu")
-		(net 29)
-	)
-	(segment
 		(start 161.8375 91.3375)
 		(end 161.8375 93)
@@
 	)
 	(segment
-		(start 168.5 92.95)
-		(end 163.55 92.95)
-		(width 0.25)
-		(layer "B.Cu")
-		(net 29)
-	)
-	(segment
 		(start 160 89.5)
 		(end 161.8375 91.3375)
@@
 		(width 0.25)
 		(layer "B.Cu")
+		(net 29)
+	)
+	(segment
+		(start 167.125 92.95)
+		(end 163.55 92.95)
+		(width 0.25)
+		(layer "B.Cu")
+		(net 29)
+	)
+	(segment
+		(start 163.55 92.95)
+		(end 163.5 93)
+		(width 0.25)
+		(layer "B.Cu")
